File: DJI_RC_N1_ESP32.kicad_sch (KiCad schematic)
At the start: 26 parts, among them J4 WE 665102131822, Q4 BSS670S2, SW1 SW_DPST, SW2 SW_DPST

Commit message: Board had been routedy
Parts:
- added J1: Conn_02x08_Odd_Even, symbol Connector_Generic:Conn_02x08_Odd_Even
- LS1: footprint Buzzer_Beeper:Buzzer_12x9.5RM7.6 -> footprints:XDCR_CMT-9605-85T
Connections:
- net GND: now also J1.1 (Pin_1), J1.2 (Pin_2), J1.3 (Pin_3), J1.4 (Pin_4), J1.5 (Pin_5), J1.6 (Pin_6)
- new net A5: J1.7 (Pin_7)
- new net DM: J1.10 (Pin_10)
- new net DP: J1.8 (Pin_8)
- new net VUSB_FRONT: J1.11 (Pin_11), J1.12 (Pin_12), J1.13 (Pin_13), J1.14 (Pin_14), J1.15 (Pin_15), J1.16 (Pin_16)
- no-connect marks 4 -> 5
Other:
- sheet Charger renamed Charger and +3V3 DCDC
- sheet Charger and +3V3 DCDC ports: added VBAT; removed none
