File: DJI_RC_N1_ESP32.kicad_sch (KiCad schematic)
At the start: 24 parts, among them J4 WE 665102131822

Commit message: Add README
Parts:
- SW_MODE1: Check_prices https://www.snapeda.com/parts/JS203011CQN/C%2526K/view-part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 -> (none); Package None -> (none); STANDARD Manufacturer Recommendations -> (none); SnapEDA_Link https://www.snapeda.com/parts/JS203011CQN/C%2526K/view-part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 -> (none)
Changed lines of the file:
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@@
 			)
 		)
-		(property "Datasheet" ""
+		(property "Datasheet" "https://www.littelfuse.com/assetdocs/littelfuse-c-k-slide-js-series-datasheet?assetguid=aba42b08-0d2c-423b-813d-a2faa5a3bb14"
 			(at 113.03 158.75 0)
 			(hide yes)
@@
 			)
 		)
-		(property "Package" "None"
-			(at 113.03 158.75 0)
-			(hide yes)
-			(show_name no)
-			(do_not_autoplace no)
-			(effects
-				(font
-					(size 1.27 1.27)
-				)
-				(justify bottom)
-			)
-		)
-		(property "Check_prices" "https://www.snapeda.com/parts/JS203011CQN/C%2526K/view-part/?ref=eda"
-			(at 113.03 158.75 0)
-			(hide yes)
-			(show_name no)
-			(do_not_autoplace no)
-			(effects
-				(font
-					(size 1.27 1.27)
-				)
-				(justify bottom)
-			)
-		)
-		(property "STANDARD" "Manufacturer Recommendations"
-			(at 113.03 158.75 0)
-			(hide yes)
-			(show_name no)
-			(do_not_autoplace no)
-			(effects
-				(font
-					(size 1.27 1.27)
-				)
-				(justify bottom)
-			)
-		)
 		(property "PARTREV" "VL"
 			(at 113.03 158.75 0)
@@
 			(at 113.03 158.75 0)
 			(hide yes)
-			(show_name no)
-			(do_not_autoplace no)
-			(effects
-				(font
-					(size 1.27 1.27)
-				)
-				(justify bottom)
-			)
-		)
-		(property "SnapEDA_Link" "https://www.snapeda.com/parts/JS203011CQN/C%2526K/view-part/?ref=snap"
-			(at 113.03 158.75 0)
-			(hide yes)

Commit message: ERC pass, Daily save
Parts:
- removed SW_LAND1: SW land, Button_Switch_SMD:SW_SPST_B3U-1000P, symbol Switch:SW_Push
- removed SW_PWR1: SW power, Button_Switch_SMD:SW_SPST_B3U-1000P, symbol Switch:SW_Push
- added Q4: BSS670S2, Package_TO_SOT_SMD:SOT-23, symbol Transistor_FET:BSS138
- added R16: TBD, Resistor_SMD:R_0603_1608Metric, symbol Device:R
- added SW1, SW2: SW_DPST, footprints:SKRPABE010, symbol Switch:SW_DPST
- LS1: footprint (none) -> Buzzer_Beeper:Buzzer_12x9.5RM7.6
Connections:
- net MODE_SW_COM_2 is gone; now on net GND: SW_MODE1.7
- net BOOT/BTN_LAND: now also SW1.2, SW1.4
- net BTN_CAM_CHANGE: no longer J4.2 (Pin_2)
- net GND: now also Q4.2 (S), SW1.1, SW1.3, SW2.1, SW2.3
- net at LS1.1: now also R16.2
- net at LS1.2: now also Q4.3 (D)
- net +3V3 renamed +3.3V
- net +3.3V: now also R16.1
- net LED1_ renamed LED_1
- net MODE_SW_CINE_1: no longer names the net of SW_MODE1.1
- net MODE_SW_COM_1: no longer names the net of SW_MODE1.3
- net MODE_SW_NORMAL_1: no longer names the net of SW_MODE1.2
- net MODE_SW_SPORT_1: no longer names the net of SW_MODE1.4
- new net BTN_PWR: SW2.2
- new net BTN_PWR_MCU: SW2.4
- new net BTN_SHOOT: J4.2 (Pin_2)
- new net BUZZER_PWM: Q4.1 (G)
- no-connect marks 0 -> 4
Other:
- moved on the sheet: LS1

Commit message: Board had been routedy
Parts:
- LS1: footprint Buzzer_Beeper:Buzzer_12x9.5RM7.6 -> footprints:XDCR_CMT-9605-85T
Changed lines of the file:
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@@
 			)
 		)
-		(property "Footprint" "Buzzer_Beeper:Buzzer_12x9.5RM7.6"
+		(property "Footprint" "footprints:XDCR_CMT-9605-85T"
 			(at 128.27 127 0)
 			(hide yes)
