File: charger.kicad_sch (KiCad schematic)
At the start: 14 parts, among them J5 USB_C_Receptacle_USB2.0_16P, Q1 BSS84, Q2 BSS670S2, U16 USBLC6-2SC6, U3 MIC5205-3.3YM5, U4 MCP73833-xxx-UN

Commit message: Board had been routedy
Parts:
- added C8: 4u7, Capacitor_SMD:C_0603_1608Metric, symbol Device:C
- added R17, R18: 5K1, Resistor_SMD:R_0603_1608Metric, symbol Device:R
Connections:
- net GND: now also C8.2, R17.2, R18.2
- net VBAT: no longer U3.1 (IN), U3.3 (EN)
- net VBAT_SWITCHED: now also U3.1 (IN), U3.3 (EN), C8.1
- net at J5.A5 (CC1): now also R18.1
- net at J5.B5 (CC2): now also R17.1
- no-connect marks 6 -> 4
